Commit message: Added madgwick filter node, IMU noise and increased the update rate

File: src/balance_bot_description/urdf/balance_bot_gazebo.urdf.xacro (robot description, xacro)
@@ -21,4 +21,5 @@
         </noise>
     </xacro:macro>
+<!--
     <xacro:property name="imu_angular_mean" value="0.0" />
     <xacro:property name="imu_angular_stddev" value="0.0" />
@@ -32,6 +33,6 @@
     <xacro:property name="imu_linear_bias_stddev" value="0.0" />
     <xacro:property name="imu_linear_dynamic_bias_stddev" value="0.0" />
-    <xacro:property name="imu_linear_dynamic_bias_correlation_time" value="0.0" />
-    <!-- <xacro:property name="imu_angular_mean" value="0.0" />
+    <xacro:property name="imu_linear_dynamic_bias_correlation_time" value="0.0" /> -->
+    <xacro:property name="imu_angular_mean" value="0.0" />
     <xacro:property name="imu_angular_stddev" value="0.00262" />
     <xacro:property name="imu_angular_bias_mean" value="0.00" />
@@ -44,9 +45,9 @@
     <xacro:property name="imu_linear_bias_stddev" value="0.147" />
     <xacro:property name="imu_linear_dynamic_bias_stddev" value="2.0e-3" />
-    <xacro:property name="imu_linear_dynamic_bias_correlation_time" value="600" /> -->
+    <xacro:property name="imu_linear_dynamic_bias_correlation_time" value="600" />
     <gazebo reference="imu_link">
         <sensor name="imu" type="imu">
             <always_on>true</always_on>
-            <update_rate>100</update_rate>
+            <update_rate>500</update_rate>
             <gz_frame_id>imu_link</gz_frame_id>
             <topic>imu</topic>
